Commit message: Changed camera

File: mir_description/urdf/include/d_camera.urdf.xacro (robot description, xacro)
@@ -11,5 +11,5 @@
         <origin xyz="0.0 0.0 0.0" rpy="0 0 0" />
         <geometry>
-          <mesh filename="package://mir_description/meshes/visual/d415.stl" />
+          <mesh filename="package://mir_description/meshes/visual/intel_r200.stl" />
         </geometry>
         <xacro:insert_block name="material_black" />
@@ -18,5 +18,5 @@
         <origin xyz="0.0 0.0 0.0" rpy="0 0 0" />
         <geometry>
-          <mesh filename="package://mir_description/meshes/visual/d415.stl" />
+          <mesh filename="package://mir_description/meshes/visual/intel_r200.stl" />
         </geometry>
       </collision>
